File: countdown_timer.brd (EAGLE design)
At the start: 65.4 x 81.3 mm, 36 parts, among them IC1 4543N, IC2 4543N, IC3 4029N, IC4 4029N, IC5 4071N, IC6 4081N, IC7 74LS32N, IC8 NE555N

Commit message: Fixed R1/R2 resistors
Eliminated pulldown resistors, routed directly to ground.
Parts:
- removed R1, R2: 10k, rcl:0204/5
Connections:
- removed net N$24: IC3.1, R1.2
- removed net N$25: IC4.1, R2.2
- net VSS: now also IC3.1, IC4.1; no longer R1.1, R2.1
Routing:
- net VSS: track 308.0 -> 330.6 mm, vias 0 -> 2
- net N$24: track 3.17 -> 0.00 mm
- net N$25: track 2.22 -> 0.00 mm
- net N$21: track 39.1 -> 37.8 mm
Changed lines of the file:
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@@
 <element name="IC6" library="40xx" package="DIL14" value="4081N" x="47.3075" y="29.845" rot="R270"/>
 <element name="IC7" library="74xx-eu" package="DIL14" value="74LS32N" x="35.2425" y="58.7375" rot="R270"/>
-<element name="R1" library="rcl" package="0204/5" value="10k" x="44.45" y="72.0725" rot="R270"/>
-<element name="R2" library="rcl" package="0204/5" value="10k" x="7.9375" y="71.12" rot="R270"/>
 <element name="R3" library="rcl" package="0204/5" value="10k" x="57.785" y="37.1475"/>
 <element name="R4" library="rcl" package="0204/5" value="22k" x="45.4025" y="76.5175"/>
@@
 <wire x1="10.16" y1="26.9875" x2="10.16" y2="24.4475" width="0.6096" layer="16"/>
 <wire x1="27.94" y1="26.9875" x2="27.94" y2="24.4475" width="0.6096" layer="16"/>
-<wire x1="7.9375" y1="48.5775" x2="15.5575" y2="48.5775" width="0.6096" layer="1"/>
+<wire x1="7.9375" y1="48.5775" x2="12.065" y2="48.5775" width="0.6096" layer="1"/>
+<wire x1="12.065" y1="48.5775" x2="15.5575" y2="48.5775" width="0.6096" layer="1"/>
 <wire x1="44.45" y1="48.5775" x2="52.07" y2="48.5775" width="0.6096" layer="1"/>
 <wire x1="52.07" y1="48.5775" x2="55.245" y2="48.5775" width="0.6096" layer="1"/>
@@
 <wire x1="39.7637" y1="72.0725" x2="39.7637" y2="72.0344" width="0.6096" layer="1"/>
 <wire x1="39.7637" y1="72.0344" x2="42.2275" y2="72.0344" width="0.6096" layer="1"/>
-<wire x1="42.2275" y1="72.0344" x2="42.2275" y2="57.4675" width="0.6096" layer="1"/>
+<wire x1="42.2275" y1="72.0344" x2="42.2275" y2="66.3575" width="0.6096" layer="1"/>
+<wire x1="42.2275" y1="66.3575" x2="42.2275" y2="57.4675" width="0.6096" layer="1"/>
 <wire x1="42.2275" y1="57.4675" x2="44.45" y2="57.4675" width="0.6096" layer="1"/>
 <wire x1="44.45" y1="57.4675" x2="44.45" y2="56.1975" width="0.6096" layer="1"/>
@@
 <wire x1="62.5475" y1="72.39" x2="62.5475" y2="55.245" width="0.6096" layer="16"/>
 <wire x1="62.5475" y1="55.245" x2="59.69" y2="55.245" width="0.6096" layer="16"/>
-<contactref element="R2" pad="1"/>
-<contactref element="R1" pad="1"/>
-<wire x1="7.9375" y1="73.66" x2="29.21" y2="70.485" width="0" layer="19" extent="1-1"/>
-<wire x1="42.2275" y1="72.0344" x2="44.45" y2="74.6125" width="0" layer="19" extent="1-1"/>
+<contactref element="IC4" pad="1"/>
+<contactref element="IC3" pad="1"/>
+<wire x1="44.45" y1="66.3575" x2="42.2275" y2="66.3575" width="0.6096" layer="1"/>
+<wire x1="7.9375" y1="66.3575" x2="8.89" y2="66.3575" width="0.4064" layer="1"/>
+<wire x1="8.89" y1="66.3575" x2="12.3825" y2="62.865" width="0.4064" layer="1"/>
+<wire x1="12.3825" y1="62.865" x2="12.3825" y2="61.2775" width="0.4064" layer="1"/>
+<via x="12.3825" y="61.2775" extent="1-16" drill="0.6" shape="square"/>
+<wire x1="12.3825" y1="61.2775" x2="12.3825" y2="56.1975" width="0.4064" layer="16"/>
+<via x="12.3825" y="56.1975" extent="1-16" drill="0.6" shape="square"/>
+<wire x1="12.3825" y1="56.1975" x2="12.3825" y2="48.895" width="0.4064" layer="1"/>
+<wire x1="12.3825" y1="48.895" x2="12.065" y2="48.5775" width="0.4064" layer="1"/>
 </signal>
 <signal name="VDD">
@@
 <contactref element="IC4" pad="14"/>
 <contactref element="IC2" pad="2"/>
-<wire x1="15.5575" y1="61.2775" x2="12.3825" y2="61.2775" width="0.4064" layer="16"/>
-<wire x1="12.3825" y1="61.2775" x2="12.3825" y2="39.6875" width="0.4064" layer="16"/>
+<wire x1="15.5575" y1="61.2775" x2="13.6525" y2="61.2775" width="0.4064" layer="16"/>
 <wire x1="12.3825" y1="39.6875" x2="10.16" y2="39.6875" width="0.4064" layer="16"/>
 <contactref element="IC5" pad="2"/>
 <wire x1="19.3675" y1="63.8175" x2="17.4625" y2="63.8175" width="0.4064" layer="16"/>
 <wire x1="17.4625" y1="63.8175" x2="17.4625" y2="65.0875" width="0.4064" layer="16"/>
-<wire x1="17.4625" y1="65.0875" x2="12.3825" y2="65.0875" width="0.4064" layer="16"/>
-<wire x1="12.3825" y1="65.0875" x2="12.3825" y2="61.2775" width="0.4064" layer="16"/>
+<wire x1="17.4625" y1="65.0875" x2="13.6525" y2="65.0875" width="0.4064" layer="16"/>
+<wire x1="13.6525" y1="65.0875" x2="13.6525" y2="61.2775" width="0.4064" layer="16"/>
+<wire x1="13.6525" y1="61.2775" x2="13.6525" y2="54.9275" width="0.4064" layer="16"/>
+<wire x1="13.6525" y1="54.9275" x2="12.3825" y2="54.9275" width="0.4064" layer="16"/>
+<wire x1="12.3825" y1="54.9275" x2="12.3825" y2="39.6875" width="0.4064" layer="16"/>
 </signal>
 <signal name="N$22">
@@
 <wire x1="19.3675" y1="67.6275" x2="19.3675" y2="66.3575" width="0.4064" layer="16"/>
 </signal>
-<signal name="N$24">
-<contactref element="R1" pad="2"/>
-<contactref element="IC3" pad="1"/>
-<wire x1="44.45" y1="69.5325" x2="44.45" y2="66.3575" width="0.4064" layer="16"/>
-</signal>
-<signal name="N$25">
-<contactref element="R2" pad="2"/>
-<contactref element="IC4" pad="1"/>
-<wire x1="7.9375" y1="66.3575" x2="7.9375" y2="68.58" width="0.4064" layer="16"/>
-</signal>
 <signal name="N$23">
