File: countdown_timer.sch (EAGLE design)
At the start: 34 parts, among them IC1 4543N, IC2 4543N, IC3 4029N, IC4 4029N, IC5 4071N, IC6 4081N, IC7 74LS32N, IC8 NE555N

Commit message: Fixed R1/R2 resistors
Eliminated pulldown resistors, routed directly to ground.
Parts:
- removed R1, R2: 10k, rcl:R-US_0204/5
Connections:
- removed net N$24: IC3A.PE, R1.2
- removed net N$25: IC4A.PE, R2.2
- net VSS: now also IC3A.PE, IC4A.PE; no longer R1.1, R2.1
Changed lines of the file:
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@@
 <part name="ONES" library="display-hp" deviceset="HD-H101" device=""/>
 <part name="TENS" library="display-hp" deviceset="HD-H101" device=""/>
-<part name="R1" library="rcl" deviceset="R-US_" device="0204/5" value="10k"/>
-<part name="R2" library="rcl" deviceset="R-US_" device="0204/5" value="10k"/>
 <part name="R3" library="rcl" deviceset="R-US_" device="0204/5" value="10k"/>
 <part name="R4" library="rcl" deviceset="R-US_" device="0204/5" value="22k"/>
@@
 <instance part="ONES" gate="M" x="93.98" y="124.46" rot="R270"/>
 <instance part="TENS" gate="M" x="93.98" y="93.98" rot="R270"/>
-<instance part="R1" gate="G$1" x="-2.54" y="116.84"/>
-<instance part="R2" gate="G$1" x="-10.16" y="78.74"/>
 <instance part="R3" gate="G$1" x="-40.64" y="111.76" rot="R90"/>
 <instance part="R4" gate="G$1" x="-78.74" y="185.42" rot="R90"/>
@@
 <wire x1="-58.42" y1="119.38" x2="-58.42" y2="106.68" width="0.1524" layer="91"/>
 <junction x="-58.42" y="106.68"/>
-<pinref part="R2" gate="G$1" pin="1"/>
 <wire x1="-15.24" y1="78.74" x2="-15.24" y2="116.84" width="0.1524" layer="91"/>
-<pinref part="R1" gate="G$1" pin="1"/>
 <wire x1="-15.24" y1="116.84" x2="-15.24" y2="119.38" width="0.1524" layer="91"/>
-<wire x1="-7.62" y1="116.84" x2="-15.24" y2="116.84" width="0.1524" layer="91"/>
 <junction x="-15.24" y="116.84"/>
 <junction x="-15.24" y="119.38"/>
+<pinref part="IC4" gate="A" pin="PE"/>
+<wire x1="-15.24" y1="78.74" x2="5.08" y2="78.74" width="0.1524" layer="91"/>
+<pinref part="IC3" gate="A" pin="PE"/>
+<wire x1="-15.24" y1="116.84" x2="5.08" y2="116.84" width="0.1524" layer="91"/>
 </segment>
 <segment>
@@
 </segment>
 </net>
-<net name="N$24" class="0">
-<segment>
-<pinref part="R1" gate="G$1" pin="2"/>
-<pinref part="IC3" gate="A" pin="PE"/>
-<wire x1="2.54" y1="116.84" x2="5.08" y2="116.84" width="0.1524" layer="91"/>
-</segment>
-</net>
-<net name="N$25" class="0">
-<segment>
-<pinref part="R2" gate="G$1" pin="2"/>
-<pinref part="IC4" gate="A" pin="PE"/>
-<wire x1="-5.08" y1="78.74" x2="5.08" y2="78.74" width="0.1524" layer="91"/>
-</segment>
-</net>
